File: steno.kicad_pcb (KiCad board)
At the start: 2 copper layers, 29 parts, among them SW1 SW_Push, SW10 SW_Push, SW11 SW_Push, SW12 SW_Push, SW13 SW_Push, SW14 SW_Push, SW15 SW_Push, SW16 SW_Push, SW17 SW_Push, SW18 SW_Push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

Commit message: Finish routing
Parts:
- A1: footprint PiPico:RaspberryPi_Pico_Common_THT -> PiPico:RaspberryPi_Pico_Common
- moved A1 0.64 mm to (130.2, 76.8)
Connections:
- A1 pad 13: Net-(A1-GND-Pad13) -> GND
- A1 pad 18: Net-(A1-GND-Pad13) -> GND
- A1 pad 23: Net-(A1-GND-Pad13) -> GND
- A1 pad 28: Net-(A1-GND-Pad13) -> GND
- A1 pad 3: Net-(A1-GND-Pad13) -> GND
- A1 pad 38: Net-(A1-GND-Pad13) -> GND
- A1 pad 8: Net-(A1-GND-Pad13) -> GND
Routing:
- net /-Z: track 0.00 -> 149.6 mm
- net /-D: track 0.00 -> 134.7 mm
- net /-S: track 0.00 -> 117.8 mm
- net /-T: track 0.00 -> 106.1 mm
- net /-G: track 0.00 -> 100.2 mm
- net /-L: track 0.00 -> 89.5 mm
- net /-B: track 0.00 -> 83.7 mm
- net /NUM2-3: track 38.1 -> 95.4 mm
- net /-P: track 17.5 -> 70.7 mm
- net /K: track 108.2 -> 99.2 mm
- net /S1: track 118.4 -> 113.5 mm
- net /T: track 87.6 -> 84.3 mm
- net /-E-: track 71.6 -> 69.7 mm
- net /-U-: track 86.2 -> 85.6 mm
- net /-O-: track 56.7 -> 57.4 mm
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- added copper zone on F.Cu, net GND
Other:
- board outline added: 247.6 x 95.3 mm
