File: steno.kicad_pcb (KiCad board)
At the start: 2 copper layers, 247.6 x 95.3 mm, 29 parts, among them SW1 SW_Push, SW10 SW_Push, SW11 SW_Push, SW12 SW_Push, SW13 SW_Push, SW14 SW_Push, SW15 SW_Push, SW16 SW_Push, SW17 SW_Push, SW18 SW_Push, SW19 SW_Push, SW2 SW_Push, SW20 SW_Push, SW21 SW_Push, SW22 SW_Push, SW23 SW_Push, SW24 SW_Push, SW25 SW_Push, SW26 SW_Push, SW27 SW_Push, SW28 SW_Push, SW3 SW_Push, SW4 SW_Push, SW5 SW_Push, SW6 SW_Push, SW7 SW_Push, SW8 SW_Push, SW9 SW_Push

Commit message: Finalized routing, added mounting holes
Parts:
- added REF**1: MountingHole_3.2mm_M3_DIN965_Pad_TopBottom, MountingHole:MountingHole_3.2mm_M3_DIN965_Pad_TopBottom, F.Cu at (22.2, 60.3)
- added REF**10: MountingHole_3.2mm_M3_DIN965_Pad_TopBottom, MountingHole:MountingHole_3.2mm_M3_DIN965_Pad_TopBottom, F.Cu at (142.9, 136.5)
- added REF**2: MountingHole_3.2mm_M3_DIN965_Pad_TopBottom, MountingHole:MountingHole_3.2mm_M3_DIN965_Pad_TopBottom, F.Cu at (98.4, 60.3)
- added REF**3: MountingHole_3.2mm_M3_DIN965_Pad_TopBottom, MountingHole:MountingHole_3.2mm_M3_DIN965_Pad_TopBottom, F.Cu at (161.9, 60.3)
- added REF**4: MountingHole_3.2mm_M3_DIN965_Pad_TopBottom, MountingHole:MountingHole_3.2mm_M3_DIN965_Pad_TopBottom, F.Cu at (257.2, 60.3)
- added REF**5: MountingHole_3.2mm_M3_DIN965_Pad_TopBottom, MountingHole:MountingHole_3.2mm_M3_DIN965_Pad_TopBottom, F.Cu at (34.9, 88.9)
- added REF**6: MountingHole_3.2mm_M3_DIN965_Pad_TopBottom, MountingHole:MountingHole_3.2mm_M3_DIN965_Pad_TopBottom, F.Cu at (244.5, 88.9)
- added REF**7: MountingHole_3.2mm_M3_DIN965_Pad_TopBottom, MountingHole:MountingHole_3.2mm_M3_DIN965_Pad_TopBottom, F.Cu at (82.5, 120.7)
- added REF**8: MountingHole_3.2mm_M3_DIN965_Pad_TopBottom, MountingHole:MountingHole_3.2mm_M3_DIN965_Pad_TopBottom, F.Cu at (177.8, 120.7)
- added REF**9: MountingHole_3.2mm_M3_DIN965_Pad_TopBottom, MountingHole:MountingHole_3.2mm_M3_DIN965_Pad_TopBottom, F.Cu at (117.5, 136.5)
- renumbered SW11 to SW10, SW22 to SW11, SW20 to SW12, SW17 to SW13, SW15 to SW14, SW12 to SW15, SW23 to SW16, SW3 to SW17, SW5 to SW18, SW7 to SW19, SW10 to SW20, SW18 to SW22, SW16 to SW23, SW13 to SW24, SW24 to SW25, SW25 to SW26, SW26 to SW27, SW27 to SW29, SW8 to SW3, SW19 to SW4, SW14 to SW5, SW1 to SW6, SW4 to SW7, SW6 to SW8
Routing:
- net /-Z: track 149.6 -> 138.5 mm
- net /W: track 73.2 -> 67.5 mm
- net /-D: track 134.7 -> 130.0 mm
- net /R: track 48.2 -> 44.7 mm
- net /K: track 99.2 -> 97.2 mm
- net /-T: track 106.1 -> 104.9 mm
- net /-L: track 89.5 -> 88.3 mm
- net /T: track 84.3 -> 84.9 mm

Commit message: Finalised design
Parts:
- added REF**: OSHW-Logo_11.4x12mm_SilkScreen, Symbol:OSHW-Logo_11.4x12mm_SilkScreen, B.Cu at (130.2, 136.5)
- added REF**9: MountingHole_3.2mm_M3_DIN965_Pad_TopBottom, MountingHole:MountingHole_3.2mm_M3_DIN965_Pad_TopBottom, F.Cu at (63.5, 136.5)
- SW1: renamed from SW2; footprint MX_2U_Modified:SW_Cherry_MX_2.00u_PCB -> MX_Modified:SW_Cherry_MX_2.00u_PCB
- SW10: renamed from SW11; footprint MX_2U_Modified:SW_Cherry_MX_2.00u_PCB -> MX_Modified:SW_Cherry_MX_2.00u_PCB
- SW11: renamed from SW12; footprint Button_Switch_Keyboard:SW_Cherry_MX_1.00u_PCB -> MX_Modified:SW_Cherry_MX_1.00u_PCB
- SW12: renamed from SW13; footprint Button_Switch_Keyboard:SW_Cherry_MX_1.00u_PCB -> MX_Modified:SW_Cherry_MX_1.00u_PCB
- SW13: renamed from SW14; footprint Button_Switch_Keyboard:SW_Cherry_MX_1.00u_PCB -> MX_Modified:SW_Cherry_MX_1.00u_PCB
- SW14: renamed from SW15; footprint Button_Switch_Keyboard:SW_Cherry_MX_1.00u_PCB -> MX_Modified:SW_Cherry_MX_1.00u_PCB
- SW15: renamed from SW16; footprint Button_Switch_Keyboard:SW_Cherry_MX_1.00u_PCB -> MX_Modified:SW_Cherry_MX_1.00u_PCB
- SW16: renamed from SW17; footprint Button_Switch_Keyboard:SW_Cherry_MX_1.00u_PCB -> MX_Modified:SW_Cherry_MX_1.00u_PCB
- SW17: renamed from SW18; footprint Button_Switch_Keyboard:SW_Cherry_MX_1.00u_PCB -> MX_Modified:SW_Cherry_MX_1.00u_PCB
- SW18: renamed from SW19; footprint Button_Switch_Keyboard:SW_Cherry_MX_1.00u_PCB -> MX_Modified:SW_Cherry_MX_1.00u_PCB
- SW19: renamed from SW20; footprint Button_Switch_Keyboard:SW_Cherry_MX_1.00u_PCB -> MX_Modified:SW_Cherry_MX_1.00u_PCB
- SW2: renamed from SW3; footprint MX_2U_Modified:SW_Cherry_MX_2.00u_PCB -> MX_Modified:SW_Cherry_MX_2.00u_PCB
- SW20: renamed from SW21; footprint Button_Switch_Keyboard:SW_Cherry_MX_1.00u_PCB -> MX_Modified:SW_Cherry_MX_1.00u_PCB
- SW21: renamed from SW22; footprint Button_Switch_Keyboard:SW_Cherry_MX_1.00u_PCB -> MX_Modified:SW_Cherry_MX_1.00u_PCB
- SW22: renamed from SW23; footprint Button_Switch_Keyboard:SW_Cherry_MX_1.00u_PCB -> MX_Modified:SW_Cherry_MX_1.00u_PCB
- SW23: renamed from SW24; footprint Button_Switch_Keyboard:SW_Cherry_MX_1.00u_PCB -> MX_Modified:SW_Cherry_MX_1.00u_PCB
- SW24: renamed from SW25; footprint Button_Switch_Keyboard:SW_Cherry_MX_1.00u_PCB -> MX_Modified:SW_Cherry_MX_1.00u_PCB
- SW25: renamed from SW26; footprint Button_Switch_Keyboard:SW_Cherry_MX_1.00u_PCB -> MX_Modified:SW_Cherry_MX_1.00u_PCB
- SW26: renamed from SW27; footprint Button_Switch_Keyboard:SW_Cherry_MX_1.00u_PCB -> MX_Modified:SW_Cherry_MX_1.00u_PCB
- SW27: renamed from SW28; footprint Button_Switch_Keyboard:SW_Cherry_MX_1.00u_PCB -> MX_Modified:SW_Cherry_MX_1.00u_PCB
- SW28: renamed from SW29; footprint Button_Switch_Keyboard:SW_Cherry_MX_1.00u_PCB -> MX_Modified:SW_Cherry_MX_1.00u_PCB
- SW3: renamed from SW4; footprint MX_2U_Modified:SW_Cherry_MX_2.00u_PCB -> MX_Modified:SW_Cherry_MX_2.00u_PCB
- SW4: renamed from SW5; footprint MX_2U_Modified:SW_Cherry_MX_2.00u_PCB -> MX_Modified:SW_Cherry_MX_2.00u_PCB
- SW5: renamed from SW6; footprint Button_Switch_Keyboard:SW_Cherry_MX_1.00u_PCB -> MX_Modified:SW_Cherry_MX_1.00u_PCB
- SW6: renamed from SW7; footprint Button_Switch_Keyboard:SW_Cherry_MX_1.00u_PCB -> MX_Modified:SW_Cherry_MX_1.00u_PCB
- SW7: renamed from SW8; footprint Button_Switch_Keyboard:SW_Cherry_MX_1.00u_PCB -> MX_Modified:SW_Cherry_MX_1.00u_PCB
- SW8: renamed from SW9; footprint Button_Switch_Keyboard:SW_Cherry_MX_1.00u_PCB -> MX_Modified:SW_Cherry_MX_1.00u_PCB
- SW9: renamed from SW10; footprint MX_2U_Modified:SW_Cherry_MX_2.00u_PCB -> MX_Modified:SW_Cherry_MX_2.00u_PCB
- moved REF**7 59.3 mm to (25.4, 136.5)
- moved REF**6 48.6 mm to (254.0, 136.5)
- moved REF**8 24.8 mm to (196.8, 136.5)
- moved REF**3 3.18 mm to (158.8, 60.3)
- moved REF**4 3.18 mm to (254.0, 60.3)
- moved REF**2 3.17 mm to (101.6, 60.3)
Routing:
- net /-B: track 83.6 -> 78.7 mm
- net /K: track 97.2 -> 93.6 mm
- net /S1: track 113.5 -> 112.9 mm
Other:
- outline, holes or cut-outs redrawn
- board text added: "nico"
- board text added: "steno"
- board text added: "v1"

Commit message: Final version
Parts:
- removed REF**5: MountingHole_3.2mm_M3_DIN965_Pad_TopBottom, MountingHole:MountingHole_3.2mm_M3_DIN965_Pad_TopBottom
Routing:
- net /T: track 84.6 -> 83.6 mm
