File: steno.kicad_sch (KiCad schematic)
At the start: 29 parts, among them SW1 SW_Push, SW10 SW_Push, SW11 SW_Push, SW12 SW_Push, SW13 SW_Push, SW14 SW_Push, SW15 SW_Push, SW16 SW_Push, SW17 SW_Push, SW18 SW_Push, SW19 SW_Push, SW2 SW_Push, SW20 SW_Push, SW21 SW_Push, SW22 SW_Push, SW23 SW_Push, SW24 SW_Push, SW25 SW_Push, SW26 SW_Push, SW27 SW_Push, SW28 SW_Push, SW3 SW_Push, SW4 SW_Push, SW5 SW_Push, SW6 SW_Push, SW7 SW_Push, SW8 SW_Push, SW9 SW_Push

Commit message: Final version
Other:
- title: Steno Keyboard -> nicosteno
Changed lines of the file:
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@@
 (kicad_sch
-	(version 20231120)
+	(version 20250114)
 	(generator "eeschema")
-	(generator_version "8.0")
+	(generator_version "9.0")
 	(paper "USLetter")
 	(title_block
-		(title "Steno Keyboard")
-		(date "2024-07-29")
-		(rev "0.1")
+		(title "nicosteno")
+		(date "2024-08-05")
+		(rev "1")
 		(company "Nicolas Landucci")
 	)
@@
 	(label "-B"
 		(at 130.81 45.72 0)
-		(fields_autoplaced yes)
 		(effects
 			(font
@@
 	(label "S1"
 		(at 48.26 135.89 0)
-		(fields_autoplaced yes)
 		(effects
 			(font
@@
 	(label "-P"
 		(at 168.91 125.73 180)
-		(fields_autoplaced yes)
 		(effects
 			(font
@@
 	(label "S1"
 		(at 85.09 38.1 180)
-		(fields_autoplaced yes)
 		(effects
 			(font
@@
 	(label "-L"
 		(at 194.31 125.73 0)
-		(fields_autoplaced yes)
 		(effects
 			(font
@@
 	(label "-S"
 		(at 204.47 135.89 180)
-		(fields_autoplaced yes)
 		(effects
 			(font
@@
 	(label "W"
 		(at 83.82 135.89 0)
-		(fields_autoplaced yes)
 		(effects
 			(font
@@
 	(label "-Z"
 		(at 130.81 71.12 0)
-		(fields_autoplaced yes)
 		(effects
 			(font
@@
 	(label "-E-"
 		(at 138.43 161.29 0)
-		(fields_autoplaced yes)
 		(effects
 			(font
@@
 	(label "-T"
 		(at 204.47 125.73 180)
-		(fields_autoplaced yes)
 		(effects
 			(font
@@
 	(label "S0"
 		(at 85.09 35.56 180)
-		(fields_autoplaced yes)
 		(effects
 			(font
@@
 	(label "STAR1"
 		(at 130.81 43.18 0)
-		(fields_autoplaced yes)
 		(effects
 			(font
@@
 	(label "STAR1"
 		(at 133.35 130.81 180)
-		(fields_autoplaced yes)
 		(effects
 			(font
@@
 	(label "STAR0"
 		(at 119.38 130.81 0)
-		(fields_autoplaced yes)
 		(effects
 			(font
@@
 	(label "NUM0-1"
 		(at 85.09 45.72 180)
-		(fields_autoplaced yes)
 		(effects
 			(font
@@
 	(label "-Z"
 		(at 229.87 135.89 0)
-		(fields_autoplaced yes)
 		(effects
 			(font
@@
 	(label "-A-"
 		(at 85.09 60.96 180)
-		(fields_autoplaced yes)
 		(effects
 			(font
@@
 	(label "H"
 		(at 85.09 53.34 180)
-		(fields_autoplaced yes)
 		(effects
 			(font
@@
 	(label "-D"
 		(at 130.81 73.66 0)
-		(fields_autoplaced yes)
 		(effects
 			(font
@@
 	(label "-P"
 		(at 130.81 48.26 0)
-		(fields_autoplaced yes)
 		(effects
 			(font
@@
 	(label "W"
 		(at 85.09 50.8 180)
-		(fields_autoplaced yes)
 		(effects
 			(font
@@
 	(label "H"
 		(at 93.98 125.73 180)
-		(fields_autoplaced yes)
 		(effects
 			(font
@@
 	(label "NUM2-3"
 		(at 177.8 115.57 0)
-		(fields_autoplaced yes)
 		(effects
 			(font
@@
 	(label "-D"
 		(at 229.87 125.73 0)
-		(fields_autoplaced yes)
 		(effects
 			(font
@@
 	(label "-U-"
 		(at 138.43 151.13 0)
-		(fields_autoplaced yes)
 		(effects
 			(font
@@
 	(label "-S"
 		(at 130.81 55.88 0)
-		(fields_autoplaced yes)
 		(effects
 			(font
@@
 	(label "-T"
 		(at 130.81 58.42 0)
-		(fields_autoplaced yes)
 		(effects
 			(font
@@
 	(label "P"
 		(at 85.09 48.26 180)
-		(fields_autoplaced yes)
 		(effects
 			(font
@@
 	(label "-E-"
 		(at 85.09 66.04 180)
-		(fields_autoplaced yes)
 		(effects
 			(font
@@
 	(label "K"
 		(at 58.42 135.89 180)
-		(fields_autoplaced yes)
 		(effects
 			(font
@@
 	(label "NUM2-3"
 		(at 130.81 68.58 0)
-		(fields_autoplaced yes)
 		(effects
 			(font
@@
 	(label "-B"
 		(at 168.91 135.89 180)
-		(fields_autoplaced yes)
 		(effects
 			(font
@@
 	(label "-G"
 		(at 194.31 135.89 0)
-		(fields_autoplaced yes)
 		(effects
 			(font
@@
 	(label "STAR0"
 		(at 85.09 58.42 180)
-		(fields_autoplaced yes)
 		(effects
 			(font
@@
 	(label "-O-"
 		(at 113.03 161.29 180)
-		(fields_autoplaced yes)
 		(effects
 			(font
@@
 	(label "-O-"
 		(at 85.09 63.5 180)
-		(fields_autoplaced yes)
 		(effects
 			(font
@@
 	(label "-L"
 		(at 130.81 53.34 0)
-		(fields_autoplaced yes)
 		(effects
 			(font
@@
 	(label "-U-"
 		(at 85.09 68.58 180)
-		(fields_autoplaced yes)
 		(effects
 			(font
@@
 	(label "T"
 		(at 85.09 40.64 180)
-		(fields_autoplaced yes)
 		(effects
 			(font
@@
 	(label "-R"
 		(at 158.75 135.89 0)
-		(fields_autoplaced yes)
 		(effects
 			(font
@@
 	(label "P"
 		(at 83.82 125.73 0)
-		(fields_autoplaced yes)
 		(effects
 			(font
@@
 	(label "S0"
 		(at 48.26 125.73 0)
-		(fields_autoplaced yes)
 		(effects
 			(font
@@
 	(label "T"
 		(at 58.42 125.73 180)
-		(fields_autoplaced yes)
 		(effects
 			(font
@@
 	(label "NUM0-1"
 		(at 67.31 115.57 0)
-		(fields_autoplaced yes)
 		(effects
 			(font
@@
 	(label "-F"
 		(at 158.75 125.73 0)
-		(fields_autoplaced yes)
 		(effects
 			(font
@@
 	(label "R"
 		(at 85.09 55.88 180)
-		(fields_autoplaced yes)
 		(effects
 			(font
@@
 	(label "R"
 		(at 93.98 135.89 180)
-		(fields_autoplaced yes)
 		(effects
 			(font
@@
 	(label "-R"
 		(at 85.09 73.66 180)
-		(fields_autoplaced yes)
 		(effects
 			(font
@@
 	(label "-A-"
 		(at 113.03 151.13 180)
-		(fields_autoplaced yes)
 		(effects
 			(font
@@
 	(label "K"
 		(at 85.09 43.18 180)
-		(fields_autoplaced yes)
 		(effects
 			(font
@@
 	(label "-G"
 		(at 130.81 50.8 0)
-		(fields_autoplaced yes)
 		(effects
 			(font
@@
 	(label "-F"
 		(at 85.09 71.12 180)
-		(fields_autoplaced yes)
 		(effects
 			(font
@@
 		)
 	)
+	(embedded_fonts no)
 )
